File: deehli_board.kicad_sch (KiCad schematic)
At the start: 44 parts, among them J1 Servo_Out, J2 PWM_In, J3 Vcc_Out, J4 DB9, J5 CAN_Ext, J6 Board_IO, SW1 SW_DPDT_x2, U1 APE1707M-50-HF, U2 LM2576HVT-5, U3 LM2576HVT-5, U4 LM2576HVT-15, U5 LD1117S33TR_SOT223, U6 LM2576HVT-15

Commit message: v1.02
Parts:
- added J7: Conn_01x08_Socket, Connector_JST:JST_EH_S8B-EH_1x08_P2.50mm_Horizontal, symbol Connector:Conn_01x08_Socket
Changed lines of the file:
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@@
+	)
+	(symbol
+		(lib_id "Connector:Conn_01x08_Socket")
+		(at 273.05 41.91 0)
+		(mirror x)
+		(unit 1)
+		(exclude_from_sim no)
+		(in_bom yes)
+		(on_board yes)
+		(dnp no)
+		(property "Reference" "J7"
+			(at 272.415 26.67 0)
+			(effects
+				(font
+					(size 1.27 1.27)
+				)
+			)
+		)
+		(property "Value" "Conn_01x08_Socket"
+			(at 272.415 29.21 0)
+			(effects
+				(font
+					(size 1.27 1.27)
+				)
+			)
+		)
+		(property "Footprint" "Connector_JST:JST_EH_S8B-EH_1x08_P2.50mm_Horizontal"
+			(at 273.05 41.91 0)
+			(effects
+				(font
+					(size 1.27 1.27)
+				)
+				(hide yes)
+			)
+		)
+		(property "Datasheet" "~"
+			(at 273.05 41.91 0)
+			(effects
+				(font
+					(size 1.27 1.27)
+				)
+				(hide yes)
+			)
+		)
+		(property "Description" "Generic connector, single row, 01x08, script generated"
+			(at 273.05 41.91 0)
+			(effects
+				(font
+					(size 1.27 1.27)
+				)
+				(hide yes)
+			)
+		)
+		(pin "3"
+		)
+		(pin "8"
+		)
+		(pin "1"
+		)
+		(pin "4"
+		)
+		(pin "7"
+		)
+		(pin "5"
+		)
+		(pin "2"
+		)
+		(pin "6"
+		)
+		(instances
+			(project ""
+				(path "/243697cf-90e5-466b-90a0-ba6eaa13d30d"
+					(reference "J7")
+					(unit 1)
+				)
+			)
+		)
 	)
 	(symbol

Commit message: vB-1.00
Parts:
- removed J4: DB9, Connector_Dsub:DSUB-9_Socket_Horizontal_P2.77x2.84mm_EdgePinOffset4.94mm_Housed_MountingHolesOffset4.94mm, symbol Connector:DE9_Socket_MountingHoles
- added J4: Conn_01x08_Socket, Connector_PinHeader_2.54mm:PinHeader_1x08_P2.54mm_Horizontal, symbol Connector:Conn_01x08_Socket
Connections:
- net 15V_ZDT: now also J7.7 (Pin_7), J4.2 (Pin_2)
- net CAN_H: now also J7.2 (Pin_2), J4.7 (Pin_7)
- net CAN_L: now also J7.1 (Pin_1), J4.8 (Pin_8)
- net GND: now also J7.8 (Pin_8), J4.1 (Pin_1)
- net at J7.3 (Pin_3): now also J4.6 (Pin_6)
- net at J7.4 (Pin_4): now also J4.5 (Pin_5)
- net at J7.5 (Pin_5): now also J4.4 (Pin_4)
- net at J7.6 (Pin_6): now also J4.3 (Pin_3)
Other:
- moved on the sheet: J7

Commit message: vB-1.01
Parts:
- C1: value Cpol 400uF -> Cpol 1000uF; footprint Capacitor_THT:CP_Radial_D6.3mm_P2.50mm -> Capacitor_THT:CP_Radial_D10.0mm_P5.00mm
- J4: value Conn_01x08_Socket -> ZDT_Pins
- J5: footprint TerminalBlock:TerminalBlock_MaiXu_MX126-5.0-03P_1x03_P5.00mm -> TerminalBlock:TerminalBlock_Xinya_XY308-2.54-3P_1x03_P2.54mm_Horizontal
- J6: footprint TerminalBlock:TerminalBlock_MaiXu_MX126-5.0-04P_1x04_P5.00mm -> TerminalBlock:TerminalBlock_Xinya_XY308-2.54-4P_1x04_P2.54mm_Horizontal
- J7: value Conn_01x08_Socket -> ZDT_Connector
Connections:
- net 15V_Other: now also C6.1, D11.1 (K), D7.2 (A), J6.1 (Pin_1), U6.2 (OUT), U6.4 (FB); no longer C7.1, D4.2 (A), D8.1 (K), J6.4 (Pin_4), U4.2 (OUT), U4.4 (FB)
- net 15V_ZDT: now also C7.1, D4.2 (A), D8.1 (K), U4.2 (OUT), U4.4 (FB); no longer C6.1, D11.1 (K), D7.2 (A), U6.2 (OUT), U6.4 (FB)
- net CAN_H: now also J6.3 (Pin_3); no longer J6.2 (Pin_2)
- net CAN_L: now also J6.4 (Pin_4); no longer J6.1 (Pin_1)
- net GND: now also J6.2 (Pin_2); no longer J6.3 (Pin_3)
Other:
- moved on the sheet: C4, C5, D1, D12, D4, D6, J6, R1, R4, R6, U1, U5

Commit message: VB-1.02
Parts:
- removed C5: Cpol 200uF, Capacitor_THT:CP_Radial_D6.3mm_P2.50mm, symbol Device:C_Polarized
- removed D12: 1N5822, Diode_THT:D_DO-201AD_P15.24mm_Horizontal, symbol Diode:1N5822
- removed J6: Board_IO, TerminalBlock:TerminalBlock_Xinya_XY308-2.54-4P_1x04_P2.54mm_Horizontal, symbol Connector:Conn_01x04_Socket
- removed JP1: Jumper_Dummy, Connector_PinHeader_2.00mm:PinHeader_1x02_P2.00mm_Vertical, symbol Jumper:Jumper_2_Small_Open
- removed U1: APE1707M-50-HF, Package_SO:SOIC-8_3.9x4.9mm_P1.27mm, symbol Regulator_Switching:APE1707M-50-HF
- added C8: 100nF, Capacitor_SMD:C_0805_2012Metric_Pad1.18x1.45mm_HandSolder, symbol Device:C
- added C9: Cpol 2x22uF, Capacitor_THT:CP_Radial_D6.3mm_P2.50mm, symbol Device:C_Polarized
- added J6: BoardPWR, TerminalBlock:TerminalBlock_Xinya_XY308-2.54-2P_1x02_P2.54mm_Horizontal, symbol Connector:Conn_01x02_Socket
- added J8: BoardCAN, TerminalBlock:TerminalBlock_Xinya_XY308-2.54-2P_1x02_P2.54mm_Horizontal, symbol Connector:Conn_01x02_Socket
- added L1, L2, L3, L4: 100u, Inductor_THT:L_Radial_D8.7mm_P5.00mm_Fastron_07HCP, symbol Device:L
- added L5: 4.7u, Inductor_THT:L_Radial_D8.7mm_P5.00mm_Fastron_07HCP, symbol Device:L
- added U1: AP63205WU, Package_TO_SOT_SMD:TSOT-23-6, symbol Regulator_Switching:AP63205WU
- J3: footprint Connector_PinHeader_2.54mm:PinHeader_1x04_P2.54mm_Vertical -> Connector_PinSocket_2.54mm:PinSocket_1x04_P2.54mm_Vertical
- J4: footprint Connector_PinHeader_2.54mm:PinHeader_1x08_P2.54mm_Horizontal -> Connector_PinSocket_2.54mm:PinSocket_1x08_P2.54mm_Horizontal
- JP2: footprint Connector_PinHeader_2.00mm:PinHeader_1x02_P2.00mm_Vertical -> Connector_PinHeader_2.54mm:PinHeader_1x02_P2.54mm_Vertical
- R5: value 15k -> 50k
Connections:
- net 15V_Other: now also J6.2 (Pin_2), L1.2, U1.2 (EN), U1.3 (IN); no longer D11.1 (K), U6.2 (OUT)
- net 15V_ZDT: now also J4.8 (Pin_8), J7.8 (Pin_8), L2.2; no longer D8.1 (K), J4.2 (Pin_2), J7.7 (Pin_7), U4.2 (OUT)
- net 5V_Other: now also C9.1, L5.2, U1.1 (FB)
- net 5V_Servo12: now also J1.7 (Pin_7), J1.8 (Pin_8), L4.2; no longer D10.1 (K), J1.5 (Pin_5), J1.6 (Pin_6), U3.2 (OUT)
- net 5V_Servo34: now also J1.5 (Pin_5), J1.6 (Pin_6), L3.2; no longer D9.1 (K), J1.7 (Pin_7), J1.8 (Pin_8), U2.2 (OUT)
- net CAN_H: now also J4.2 (Pin_2), J8.1 (Pin_1); no longer J4.7 (Pin_7)
- net CAN_L: now also J4.1 (Pin_1), J8.2 (Pin_2); no longer J4.8 (Pin_8)
- net GND: now also J4.7 (Pin_7), J7.7 (Pin_7), C9.2, J6.1 (Pin_1), U1.4 (GND); no longer J4.1 (Pin_1), J7.8 (Pin_8)
- net at C1.1, SW1.2 (B), U2.1 (VIN)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: no longer R5.2
- net at PWR_IN1.1, PWR_IN2.1 (Pin_1), SW1.3 (C): now also R5.2
- net at J7.3 (Pin_3): now also J4.3 (Pin_3); no longer J4.6 (Pin_6)
- net at J7.4 (Pin_4): now also J4.4 (Pin_4); no longer J4.5 (Pin_5)
- net at J7.5 (Pin_5): now also J4.5 (Pin_5); no longer J4.4 (Pin_4)
- net at J7.6 (Pin_6): now also J4.6 (Pin_6); no longer J4.3 (Pin_3)
- new net: D8.1 (K), L2.1, U4.2 (OUT)
- new net: D10.1 (K), L4.1, U3.2 (OUT)
- new net: D11.1 (K), L1.1, U6.2 (OUT)
- new net: C8.1, U1.6 (BST)
- new net: C8.2, L5.1, U1.5 (SW)
- new net: D9.1 (K), L3.1, U2.2 (OUT)
Other:
- moved on the sheet: C2, C3, C4, C6, C7, D1, D11, D2, D3, D4, D5, D6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
